File: daemonbite_controller_hub/daemonbite_controller_hub.kicad_pcb (KiCad board)
At the start: 2 copper layers, 106.9 x 68.7 mm, 12 parts, among them J1 Conn_01x01, J2 Conn_01x01, J3 Conn_01x01, J4 Conn_01x01, U1 ATmega32u4, U2 ATmega32u4, U3 SNES_port, U4 SNES_port, U5 NES_port, U6 NES_port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

Commit message: Add files via upload
Parts:
- U1, U2: footprint daemonbite:ATmega32U4 -> daemonbite_controller_hub:ATmega32U4
- U3, U4: footprint daemonbite:SNES_port -> daemonbite_controller_hub:SNES_port
- U5, U6: footprint daemonbite:NES_port -> daemonbite_controller_hub:NES_port
- U7, U8: footprint daemonbite:DSUB-9_Male_Horizontal_P2.77x2.84mm_EdgePinOffset7.70mm_Housed_MountingHolesOffset9.12mm -> daemonbite_controller_hub:DSUB-9_Male_Horizontal_P2.77x2.84mm_EdgePinOffset7.70mm_Housed_MountingHolesOffset9.12mm
