File: daemonbite_controller_hub/daemonbite_controller_hub.kicad_sch (KiCad schematic)
At the start: 12 parts, among them J1 Conn_01x01, J2 Conn_01x01, J3 Conn_01x01, J4 Conn_01x01, U1 ATmega32u4, U2 ATmega32u4, U3 SNES_port, U4 SNES_port, U5 NES_port, U6 NES_port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

Commit message: Add files via upload
Parts:
- U1, U2: footprint daemonbite:ATmega32U4 -> daemonbite_controller_hub:ATmega32U4
- U3, U4: footprint daemonbite:SNES_port -> daemonbite_controller_hub:SNES_port
- U5, U6: footprint daemonbite:NES_port -> daemonbite_controller_hub:NES_port
- U7, U8: footprint daemonbite:DSUB-9_Male_Horizontal_P2.77x2.84mm_EdgePinOffset7.70mm_Housed_MountingHolesOffset9.12mm -> daemonbite_controller_hub:DSUB-9_Male_Horizontal_P2.77x2.84mm_EdgePinOffset7.70mm_Housed_MountingHolesOffset9.12mm
Changed lines of the file:
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@@
       (effects (font (size 1.27 1.27)) (justify left))
     )
-    (property "Footprint" "daemonbite:DSUB-9_Male_Horizontal_P2.77x2.84mm_EdgePinOffset7.70mm_Housed_MountingHolesOffset9.12mm" (id 2) (at 195.58 81.28 0)
+    (property "Footprint" "daemonbite_controller_hub:DSUB-9_Male_Horizontal_P2.77x2.84mm_EdgePinOffset7.70mm_Housed_MountingHolesOffset9.12mm" (id 2) (at 195.58 81.28 0)
       (effects (font (size 1.27 1.27)) hide)
     )
@@
       (effects (font (size 1.27 1.27)) (justify left))
     )
-    (property "Footprint" "daemonbite:DSUB-9_Male_Horizontal_P2.77x2.84mm_EdgePinOffset7.70mm_Housed_MountingHolesOffset9.12mm" (id 2) (at 257.81 78.74 0)
+    (property "Footprint" "daemonbite_controller_hub:DSUB-9_Male_Horizontal_P2.77x2.84mm_EdgePinOffset7.70mm_Housed_MountingHolesOffset9.12mm" (id 2) (at 257.81 78.74 0)
       (effects (font (size 1.27 1.27)) hide)
     )
@@
       (effects (font (size 1.27 1.27)) (justify left))
     )
-    (property "Footprint" "daemonbite:SNES_port" (id 2) (at 38.1 81.28 0)
+    (property "Footprint" "daemonbite_controller_hub:SNES_port" (id 2) (at 38.1 81.28 0)
       (effects (font (size 1.27 1.27)) hide)
     )
@@
       (effects (font (size 1.27 1.27)) (justify left))
     )
-    (property "Footprint" "daemonbite:SNES_port" (id 2) (at 78.74 81.28 0)
+    (property "Footprint" "daemonbite_controller_hub:SNES_port" (id 2) (at 78.74 81.28 0)
       (effects (font (size 1.27 1.27)) hide)
     )
@@
       (effects (font (size 1.27 1.27)) (justify left))
     )
-    (property "Footprint" "daemonbite:NES_port" (id 2) (at 106.68 81.28 0)
+    (property "Footprint" "daemonbite_controller_hub:NES_port" (id 2) (at 106.68 81.28 0)
       (effects (font (size 1.27 1.27)) hide)
     )
@@
       (effects (font (size 1.27 1.27)) (justify left))
     )
-    (property "Footprint" "daemonbite:NES_port" (id 2) (at 134.62 81.28 0)
+    (property "Footprint" "daemonbite_controller_hub:NES_port" (id 2) (at 134.62 81.28 0)
       (effects (font (size 1.27 1.27)) hide)
     )
@@
     (property "Reference" "U1" (id 0) (at 43.815 21.209 0))
     (property "Value" "ATmega32u4" (id 1) (at 43.815 23.5204 0))
-    (property "Footprint" "daemonbite:ATmega32U4" (id 2) (at 44.45 34.29 0)
+    (property "Footprint" "daemonbite_controller_hub:ATmega32U4" (id 2) (at 44.45 34.29 0)
       (effects (font (size 1.27 1.27)) hide)
     )
@@
     (property "Reference" "U2" (id 0) (at 231.775 19.939 0))
     (property "Value" "ATmega32u4" (id 1) (at 231.775 22.2504 0))
-    (property "Footprint" "daemonbite:ATmega32U4" (id 2) (at 232.41 33.02 0)
+    (property "Footprint" "daemonbite_controller_hub:ATmega32U4" (id 2) (at 232.41 33.02 0)
       (effects (font (size 1.27 1.27)) hide)
     )
@@
     )
     (path "/00000000-0000-0000-0000-000060185ba2"
-      (reference "U1") (unit 1) (value "ATmega32u4") (footprint "daemonbite:ATmega32U4")
+      (reference "U1") (unit 1) (value "ATmega32u4") (footprint "daemonbite_controller_hub:ATmega32U4")
     )
     (path "/00000000-0000-0000-0000-0000601e3dc4"
-      (reference "U2") (unit 1) (value "ATmega32u4") (footprint "daemonbite:ATmega32U4")
+      (reference "U2") (unit 1) (value "ATmega32u4") (footprint "daemonbite_controller_hub:ATmega32U4")
     )
     (path "/00000000-0000-0000-0000-00006018a475"
-      (reference "U3") (unit 1) (value "SNES_port") (footprint "daemonbite:SNES_port")
+      (reference "U3") (unit 1) (value "SNES_port") (footprint "daemonbite_controller_hub:SNES_port")
     )
     (path "/00000000-0000-0000-0000-00006018ae31"
-      (reference "U4") (unit 1) (value "SNES_port") (footprint "daemonbite:SNES_port")
+      (reference "U4") (unit 1) (value "SNES_port") (footprint "daemonbite_controller_hub:SNES_port")
     )
     (path "/00000000-0000-0000-0000-0000601993be"
-      (reference "U5") (unit 1) (value "NES_port") (footprint "daemonbite:NES_port")
+      (reference "U5") (unit 1) (value "NES_port") (footprint "daemonbite_controller_hub:NES_port")
     )
     (path "/00000000-0000-0000-0000-0000601993b8"
-      (reference "U6") (unit 1) (value "NES_port") (footprint "daemonbite:NES_port")
+      (reference "U6") (unit 1) (value "NES_port") (footprint "daemonbite_controller_hub:NES_port")
     )
     (path "/00000000-0000-0000-0000-0000606d6f77"
-      (reference "U7") (unit 1) (value "MD_port") (footprint "daemonbite:DSUB-9_Male_Horizontal_P2.77x2.84mm_EdgePinOffset7.70mm_Housed_MountingHolesOffset9.12mm")
+      (reference "U7") (unit 1) (value "MD_port") (footprint "daemonbite_controller_hub:DSUB-9_Male_Horizontal_P2.77x2.84mm_EdgePinOffset7.70mm_Housed_MountingHolesOffset9.12mm")
     )
     (path "/00000000-0000-0000-0000-0000606d672b"
-      (reference "U8") (unit 1) (value "MD_port") (footprint "daemonbite:DSUB-9_Male_Horizontal_P2.77x2.84mm_EdgePinOffset7.70mm_Housed_MountingHolesOffset9.12mm")
-    )
-  )
+      (reference "U8") (unit 1) (value "MD_port") (footprint "daemonbite_controller_hub:DSUB-9_Male_Horizontal_P2.77x2.84mm_EdgePinOffset7.70mm_Housed_MountingHolesOffset9.12mm")
+    )
+  )
